File: pcb/orch.kicad_pcb (KiCad board)
At the start: 2 copper layers, 134 parts, among them J1 AVR-ISP-6, P1 USB_C_Receptacle_USB2.0, SW1 MX-NoLED, SW10 MX-NoLED, SW11 MX-NoLED, SW12 MX-NoLED, SW13 MX-NoLED, SW14 MX-NoLED, SW15 MX-NoLED, SW16 MX-NoLED, SW17 MX-NoLED, SW18 MX-NoLED, SW19 MX-NoLED, SW2 MX-NoLED, SW20 MX-NoLED, SW21 MX-NoLED, SW22 MX-NoLED, SW23 MX-NoLED, SW24 MX-NoLED, SW25 MX-NoLED, SW26 MX-NoLED, SW27 MX-NoLED, SW28 MX-NoLED, SW29 MX-NoLED, SW3 MX-NoLED, SW30 MX-NoLED, SW31 MX-NoLED, SW32 MX-NoLED, SW33 MX-NoLED, SW34 MX-NoLED, SW35 MX-NoLED, SW36 MX-NoLED, SW37 MX-NoLED, SW38 MX-NoLED, SW39 MX-NoLED, SW4 MX-NoLED, SW40 MX-NoLED, SW41 MX-NoLED, SW42 MX-NoLED, SW43 MX-NoLED, SW44 MX-NoLED, SW45 MX-NoLED, SW46 MX-NoLED, SW47 MX-NoLED, SW48 MX-NoLED, SW49 MX-NoLED, SW5 MX-NoLED, SW50 MX-NoLED, SW51 MX-NoLED, SW52 MX-NoLED, SW53 MX-NoLED, SW54 MX-NoLED, SW55 MX-NoLED, SW56 MX-NoLED, SW57 MX-NoLED, SW58 Reset, SW6 MX-NoLED, SW7 MX-NoLED, SW8 MX-NoLED, SW9 MX-NoLED, U1 ATmega32U4-AU, Y1 16MHz

Commit message: pcb done
Parts:
- D1, D10, D11, D12, D13, D14, D15, D16, D17, D18, D19, D2, D20, D21, D22, D23, D24, D25, D26, D27, D28, D29, D3, D30, D31, D32, D33, D34, D35, D36, D37, D38, D39, D4, D40, D41, D42, D43, D44, D45, D46, D47, D48, D49, D5, D50, D51, D52, D53, D54, D55, D56, D57, D6, D7, D8, D9: footprint Diode_SMD:D_0805_2012Metric_Pad1.15x1.40mm_HandSolder -> orch:D_DO-35_SOD27_P5.08mm_Horizontal
- moved R3 49.0 mm to (310.5, 86.9), turned to 90 degrees
- moved R2 48.7 mm to (313.9, 86.9), turned to 90 degrees
- moved C2 45.7 mm to (322.6, 121.6), turned to 225 degrees
- moved C7 45.7 mm to (288.1, 74.8), turned to 90 degrees
- moved C6 44.6 mm to (284.6, 74.8), turned to 90 degrees
- moved C3 44.1 mm to (274.2, 74.8), turned to 90 degrees
- moved C5 43.8 mm to (281.1, 74.8), turned to 90 degrees
- moved C4 43.5 mm to (277.6, 74.8), turned to 90 degrees
- moved C1 42.9 mm to (326.1, 118.1), turned to 225 degrees
- moved Y1 38.9 mm to (320.9, 116.3), turned to 45 degrees
- moved J1 36.1 mm to (319.8, 94.5), turned to 180 degrees
- moved R1 33.9 mm to (332.2, 94.5), turned to 270 degrees
- moved R4 30.7 mm to (288.8, 64.5)
- moved F1 28.8 mm to (320.5, 78.8)
- moved SW58 27.9 mm to (326.8, 94.5)
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Connections:
- D53 pad 1: /Row2 -> /Row4
- U1 pad 18: /Col13 -> /Col11
- U1 pad 20: /Col11 -> /Col13
Routing:
- net /Col1: track 0.00 -> 321.2 mm, vias 0 -> 1
- net /Col2: track 0.00 -> 301.5 mm, vias 0 -> 1
- net /Row3: track 0.00 -> 291.3 mm
- net /Row2: track 0.00 -> 287.4 mm
- net /Row4: track 0.00 -> 287.3 mm
- net /Row1: track 0.00 -> 286.7 mm
- net /Col3: track 0.00 -> 283.7 mm, vias 0 -> 1
- net /Col4: track 0.00 -> 262.8 mm, vias 0 -> 1
- net /Col5: track 0.00 -> 241.6 mm, vias 0 -> 1
- net /Col6: track 0.00 -> 217.0 mm, vias 0 -> 1
- net /Col8: track 0.00 -> 186.3 mm, vias 0 -> 1
- net /Col7: track 0.00 -> 186.2 mm, vias 0 -> 1
- net /Col9: track 0.00 -> 170.4 mm, vias 0 -> 1
- net /Col11: track 0.00 -> 157.7 mm
- net /Col10: track 0.00 -> 152.3 mm, vias 0 -> 1
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- added copper zone on B.Cu, net GND
- added copper zone on F.Cu, net GND
Other:
- board outline added: 313.6 x 80.8 mm
- rule trace_min: 0.2 -> 0.25
- rule via_min_drill: 0.3 -> 0.254
- rule via_min_size: 0.4 -> 0.381

Commit message: v0.0.1
Parts:
- added D58: SK6812, LED_SMD:LED_SK6812_PLCC4_5.0x5.0mm_P3.2mm, B.Cu at (294.9, 95.8)
- added D59: SK6812, LED_SMD:LED_SK6812_PLCC4_5.0x5.0mm_P3.2mm, B.Cu at (251.0, 95.8)
- added D60: SK6812, LED_SMD:LED_SK6812_PLCC4_5.0x5.0mm_P3.2mm, B.Cu at (181.1, 95.8)
- added D61: SK6812, LED_SMD:LED_SK6812_PLCC4_5.0x5.0mm_P3.2mm, B.Cu at (121.2, 95.8)
- added D62: SK6812, LED_SMD:LED_SK6812_PLCC4_5.0x5.0mm_P3.2mm, B.Cu at (78.2, 95.8)
Connections:
- U1 pad 18: /Col11 -> /Col13
- U1 pad 20: /Col13 -> /Col11
- U1 pad 40: Net-(U1-Pad40) -> /RGB
Routing:
- net +5V: track 146.1 -> 411.1 mm, vias 2 -> 12
- net /Col3: track 283.7 -> 364.6 mm
- net /Col5: track 241.6 -> 320.2 mm
- net /Col6: track 217.0 -> 295.5 mm
- net Net-(D59-Pad4): track 0.00 -> 66.3 mm, vias 0 -> 2
- net Net-(D60-Pad4): track 0.00 -> 56.4 mm, vias 0 -> 2
- net /Col8: track 186.3 -> 239.8 mm
- net Net-(D58-Pad4): track 0.00 -> 40.5 mm, vias 0 -> 2
- net Net-(D61-Pad4): track 0.00 -> 39.4 mm, vias 0 -> 2
- net /Col4: track 262.8 -> 279.2 mm
- net /Col2: track 301.5 -> 315.5 mm
- net /RGB: track 0.00 -> 12.0 mm
- net /Col7: track 186.2 -> 196.8 mm
- net Net-(P1-PadA6): track 24.4 -> 26.1 mm
- net Net-(P1-PadA7): track 23.3 -> 25.0 mm
Other:
- rule trace_min: 0.25 -> 0.2
- board text added: "orch v0.0.1"

Commit message: clean up pages
Parts:
- moved D22 51.2 mm to (164.4, 134.6)
- moved D23 51.2 mm to (164.4, 153.6)
- moved D24 51.2 mm to (173.9, 172.6)
- moved D26 51.2 mm to (183.4, 134.6)
- moved D27 51.2 mm to (183.4, 153.6)
- moved D29 51.2 mm to (202.4, 134.6)
- moved D30 51.2 mm to (202.4, 153.6)
- moved D31 51.2 mm to (202.4, 172.6)
- moved D33 51.2 mm to (221.4, 134.6)
- moved D34 51.2 mm to (221.4, 153.6)
- moved D35 51.2 mm to (223.8, 172.6)
- moved D37 51.2 mm to (240.4, 134.6)
- moved D38 51.2 mm to (240.4, 153.6)
- moved D39 51.2 mm to (245.2, 172.6)
- moved D4 51.2 mm to (64.7, 172.6)
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