File: pcb/orch.sch (KiCad schematic (older format))
At the start: 29 parts, among them J1 AVR-ISP-6, P1 USB_C_Receptacle_USB2.0, SW1 MX-NoLED, SW2 MX-NoLED, SW3 MX-NoLED, SW4 MX-NoLED, SW7 Reset, SW8 Boot, U1 ATmega32U4-AU, Y1 16MHz

Commit message: pcb layout
Parts:
- removed H19, H20, H21, H22: MountingHole, MountingHole:MountingHole_2.2mm_M2, symbol Mechanical:MountingHole
- removed SW8: Boot, Button_Switch_THT:SW_PUSH_6mm_H4.3mm, symbol Switch:SW_Push
- added C8: 1u, Capacitor_SMD:C_0805_2012Metric_Pad1.15x1.40mm_HandSolder, symbol Device:C
- added D10, D11, D12, D14, D15, D16, D17, D18, D19, D2, D20, D21, D22, D23, D24, D25, D26, D27, D28, D29, D3, D30, D31, D32, D33, D34, D35, D36, D37, D38, D39, D4, D40, D41, D42, D43, D44, D45, D46, D47, D48, D49, D50, D51, D52, D53, D54, D55, D56, D57, D6, D7, D8: 1N4148, Diode_SMD:D_0805_2012Metric_Pad1.15x1.40mm_HandSolder, symbol Device:D
- added R4, R5: 5.1k, Resistor_SMD:R_0805_2012Metric_Pad1.15x1.40mm_HandSolder, symbol Device:R
- added R6: 10K, Resistor_SMD:R_0805_2012Metric_Pad1.15x1.40mm_HandSolder, symbol Device:R
- added SW10, SW11, SW12, SW14, SW15, SW17, SW18, SW19, SW20, SW21, SW22, SW23, SW25, SW26, SW27, SW28, SW29, SW30, SW31, SW32, SW33, SW34, SW36, SW37, SW38, SW39, SW4, SW40, SW41, SW42, SW43, SW44, SW45, SW47, SW48, SW50, SW51, SW53, SW54, SW55, SW56, SW57, SW6, SW7, SW8: MX-NoLED, orch:MX-1U-NoLED, symbol orch:MX-NoLED
- added SW16, SW35, SW46: MX-NoLED, orch:MX-1.25U-NoLED, symbol orch:MX-NoLED
- added SW2, SW3: MX-NoLED, orch:MX-1.75U-NoLED, symbol orch:MX-NoLED
- added SW24: MX-NoLED, orch:MX-2U-NoLED, symbol orch:MX-NoLED
- added SW49: MX-NoLED, orch:MX-2.25U-NoLED, symbol orch:MX-NoLED
- added SW52: MX-NoLED, orch:MX-1.5U-NoLED, symbol orch:MX-NoLED
- C1, C2, C4, C5, C6, C7: footprint Capacitor_THT:C_Rect_L4.0mm_W2.5mm_P2.50mm -> Capacitor_SMD:C_0805_2012Metric_Pad1.15x1.40mm_HandSolder
- C3: footprint Capacitor_THT:C_Radial_D4.0mm_H7.0mm_P1.50mm -> Capacitor_SMD:C_0805_2012Metric_Pad1.15x1.40mm_HandSolder
- D1: footprint pin-check:D_DO-35_SOD27_P5.08mm_Horizontal -> Diode_SMD:D_0805_2012Metric_Pad1.15x1.40mm_HandSolder
- D13: renamed from D4; footprint pin-check:D_DO-35_SOD27_P5.08mm_Horizontal -> Diode_SMD:D_0805_2012Metric_Pad1.15x1.40mm_HandSolder
- D5: renamed from D2; footprint pin-check:D_DO-35_SOD27_P5.08mm_Horizontal -> Diode_SMD:D_0805_2012Metric_Pad1.15x1.40mm_HandSolder
- D9: renamed from D3; footprint pin-check:D_DO-35_SOD27_P5.08mm_Horizontal -> Diode_SMD:D_0805_2012Metric_Pad1.15x1.40mm_HandSolder
- F1: footprint (none) -> Fuse:Fuse_0805_2012Metric_Pad1.15x1.40mm_HandSolder
- J1: footprint Connector_PinHeader_2.54mm:PinHeader_2x03_P2.54mm_Vertical -> Connector:Tag-Connect_TC2030-IDC-NL_2x03_P1.27mm_Vertical
- P1: footprint pin-check:USB_C_GCT_USB4085 -> orch:USB_C_GCT_USB4085
- R1: footprint Resistor_THT:R_Axial_DIN0204_L3.6mm_D1.6mm_P7.62mm_Horizontal -> Resistor_SMD:R_0805_2012Metric_Pad1.15x1.40mm_HandSolder
- R2, R3: footprint (none) -> Resistor_SMD:R_0805_2012Metric_Pad1.15x1.40mm_HandSolder
- SW1: footprint pin-check:MX-1U-NoLED -> orch:MX-1.5U-NoLED; symbol pin-check:MX-NoLED -> orch:MX-NoLED
- SW13: renamed from SW4; footprint pin-check:MX-1U-NoLED -> orch:MX-1U-NoLED; symbol pin-check:MX-NoLED -> orch:MX-NoLED
- SW5: renamed from SW2; footprint pin-check:MX-1U-NoLED -> orch:MX-1U-NoLED; symbol pin-check:MX-NoLED -> orch:MX-NoLED
- SW58: renamed from SW7; footprint Button_Switch_THT:SW_PUSH_6mm_H4.3mm -> Button_Switch_SMD:SW_Push_1P1T_NO_CK_KMR2
- SW9: renamed from SW3; footprint pin-check:MX-1U-NoLED -> orch:MX-1U-NoLED; symbol pin-check:MX-NoLED -> orch:MX-NoLED
- Y1: footprint Crystal:Crystal_HC49-4H_Vertical -> Crystal:Crystal_SMD_Abracon_ABM3-2Pin_5.0x3.2mm_HandSoldering
Connections:
- net labels added: Col1, Col10, Col11, Col12, Col13, Col14, Col15, Col2, Col3, Col4, Col5, Col6, Col7, Col8, Col9, D+, MISO, MOSI, Row1, Row2, Row3, Row4, SCK, XTAL1, XTAL2
- net labels removed: ColA, ColAExt, ColB, ColBExt, ColC, ColCExt, ColD, ColDExt, D5, Row0, Row0Ext
- wire segments 74 -> 187
- no-connect marks 2 -> 10
Other:
- note added: "Crystal"
- note added: "ISP Header"
- note added: "Microcontroller"
- note added: "Reset Switch"
- note removed: "Boot and Reset Switches"
- note removed: "Microcontroller, Crystal, and ISP Headers"
- note removed: "Mounting Holes"

Commit message: pcb done
Parts:
- D1, D10, D11, D12, D13, D14, D15, D16, D17, D18, D19, D2, D20, D21, D22, D23, D24, D25, D26, D27, D28, D29, D3, D30, D31, D32, D33, D34, D35, D36, D37, D38, D39, D4, D40, D41, D42, D43, D44, D45, D46, D47, D48, D49, D5, D50, D51, D52, D53, D54, D55, D56, D57, D6, D7, D8, D9: footprint Diode_SMD:D_0805_2012Metric_Pad1.15x1.40mm_HandSolder -> orch:D_DO-35_SOD27_P5.08mm_Horizontal

Commit message: v0.0.1
Parts:
- added D58, D59, D60, D61, D62: SK6812, LED_SMD:LED_SK6812_PLCC4_5.0x5.0mm_P3.2mm, symbol LED:SK6812
Connections:
- net labels added: RGB
- wire segments 187 -> 201
- no-connect marks 10 -> 9
Changed lines of the file:
@@
 Col10
 Text Label 2350 3000 0    50   ~ 0
-Col13
+Col11
 Text Label 2350 2900 0    50   ~ 0
 Col12
 Text Label 2350 2800 0    50   ~ 0
-Col11
+Col13
 Text Label 2350 2300 0    50   ~ 0
 Col14
 Text Label 2350 4000 0    50   ~ 0
 Col15
-NoConn ~ 2350 4100
 NoConn ~ 2350 4200
 NoConn ~ 2350 4300
@@
 	8950 9300 8950 11100
 Connection ~ 8950 9300
+$Comp
+L LED:SK6812 D60
+U 1 1 60043709
+P 5900 4400
+F 0 "D60" H 6244 4446 50  0000 L CNN
+F 1 "SK6812" H 6244 4355 50  0000 L CNN
+F 2 "LED_SMD:LED_SK6812_PLCC4_5.0x5.0mm_P3.2mm" H 5950 4100 50  0001 L TNN
+F 3 "https://cdn-shop.adafruit.com/product-files/1138/SK6812+LED+datasheet+.pdf" H 6000 4025 50  0001 L TNN
+	1    5900 4400
+	1    0    0    -1
+$EndComp
+$Comp
+L LED:SK6812 D59
+U 1 1 6004455E
+P 4850 4400
+F 0 "D59" H 5194 4446 50  0000 L CNN
+F 1 "SK6812" H 5194 4355 50  0000 L CNN
+F 2 "LED_SMD:LED_SK6812_PLCC4_5.0x5.0mm_P3.2mm" H 4900 4100 50  0001 L TNN
+F 3 "https://cdn-shop.adafruit.com/product-files/1138/SK6812+LED+datasheet+.pdf" H 4950 4025 50  0001 L TNN
+	1    4850 4400
+	1    0    0    -1
+$EndComp
+$Comp
+L LED:SK6812 D58
+U 1 1 600451BB
+P 3800 4400
+F 0 "D58" H 4144 4446 50  0000 L CNN
+F 1 "SK6812" H 4144 4355 50  0000 L CNN
+F 2 "LED_SMD:LED_SK6812_PLCC4_5.0x5.0mm_P3.2mm" H 3850 4100 50  0001 L TNN
+F 3 "https://cdn-shop.adafruit.com/product-files/1138/SK6812+LED+datasheet+.pdf" H 3900 4025 50  0001 L TNN
+	1    3800 4400
+	1    0    0    -1
+$EndComp
+$Comp
+L LED:SK6812 D61
+U 1 1 600459D4
+P 6950 4400
+F 0 "D61" H 7294 4446 50  0000 L CNN
+F 1 "SK6812" H 7294 4355 50  0000 L CNN
+F 2 "LED_SMD:LED_SK6812_PLCC4_5.0x5.0mm_P3.2mm" H 7000 4100 50  0001 L TNN
+F 3 "https://cdn-shop.adafruit.com/product-files/1138/SK6812+LED+datasheet+.pdf" H 7050 4025 50  0001 L TNN
+	1    6950 4400
+	1    0    0    -1
+$EndComp
+$Comp
+L LED:SK6812 D62
+U 1 1 60047365
+P 8000 4400
+F 0 "D62" H 8344 4446 50  0000 L CNN
+F 1 "SK6812" H 8344 4355 50  0000 L CNN
+F 2 "LED_SMD:LED_SK6812_PLCC4_5.0x5.0mm_P3.2mm" H 8050 4100 50  0001 L TNN
+F 3 "https://cdn-shop.adafruit.com/product-files/1138/SK6812+LED+datasheet+.pdf" H 8100 4025 50  0001 L TNN
+	1    8000 4400
+	1    0    0    -1
+$EndComp
+Text Label 2350 4100 0    50   ~ 0
+RGB
+$Comp
+L power:+5V #PWR02
+U 1 1 6005462B
+P 3800 4000
+F 0 "#PWR02" H 3800 3850 50  0001 C CNN
+F 1 "+5V" H 3815 4173 50  0000 C CNN
+F 2 "" H 3800 4000 50  0001 C CNN
+F 3 "" H 3800 4000 50  0001 C CNN
+	1    3800 4000
+	1    0    0    -1
+$EndComp
+Wire Wire Line
+	3800 4100 3800 4000
+Wire Wire Line
+	3800 4100 4850 4100
+Connection ~ 3800 4100
+Connection ~ 4850 4100
+Wire Wire Line
+	4850 4100 5900 4100
+Connection ~ 5900 4100
+Wire Wire Line
+	5900 4100 6950 4100
+Connection ~ 6950 4100
+Wire Wire Line
+	6950 4100 8000 4100
+$Comp
+L power:GND #PWR03
+U 1 1 6006B048
+P 3800 4800
+F 0 "#PWR03" H 3800 4550 50  0001 C CNN
+F 1 "GND" H 3805 4627 50  0000 C CNN
+F 2 "" H 3800 4800 50  0001 C CNN
+F 3 "" H 3800 4800 50  0001 C CNN
+	1    3800 4800
+	1    0    0    -1
+$EndComp
+Wire Wire Line
+	3800 4700 3800 4800
+Wire Wire Line
+	3800 4700 4850 4700
+Connection ~ 3800 4700
+Connection ~ 4850 4700
+Wire Wire Line
+	4850 4700 5900 4700
+Connection ~ 5900 4700
+Wire Wire Line
+	5900 4700 6950 4700
+Connection ~ 6950 4700
+Wire Wire Line
+	6950 4700 8000 4700
+Text Label 3500 4400 2    50   ~ 0
+RGB
+Wire Wire Line
+	4100 4400 4550 4400
+Wire Wire Line
+	5150 4400 5600 4400
+Wire Wire Line
+	6200 4400 6650 4400
+Wire Wire Line
+	7250 4400 7700 4400
 $EndSCHEMATC

Commit message: clean up pages
Other:
- note added: "RGB LEDs"
