File: pcb/orch.sch (KiCad schematic (older format))
At the start: 139 parts, among them J1 AVR-ISP-6, P1 USB_C_Receptacle_USB2.0, SW1 MX-NoLED, SW10 MX-NoLED, SW11 MX-NoLED, SW12 MX-NoLED, SW13 MX-NoLED, SW14 MX-NoLED, SW15 MX-NoLED, SW16 MX-NoLED, SW17 MX-NoLED, SW18 MX-NoLED, SW19 MX-NoLED, SW2 MX-NoLED, SW20 MX-NoLED, SW21 MX-NoLED, SW22 MX-NoLED, SW23 MX-NoLED, SW24 MX-NoLED, SW25 MX-NoLED, SW26 MX-NoLED, SW27 MX-NoLED, SW28 MX-NoLED, SW29 MX-NoLED, SW3 MX-NoLED, SW30 MX-NoLED, SW31 MX-NoLED, SW32 MX-NoLED, SW33 MX-NoLED, SW34 MX-NoLED, SW35 MX-NoLED, SW36 MX-NoLED, SW37 MX-NoLED, SW38 MX-NoLED, SW39 MX-NoLED, SW4 MX-NoLED, SW40 MX-NoLED, SW41 MX-NoLED, SW42 MX-NoLED, SW43 MX-NoLED, SW44 MX-NoLED, SW45 MX-NoLED, SW46 MX-NoLED, SW47 MX-NoLED, SW48 MX-NoLED, SW49 MX-NoLED, SW5 MX-NoLED, SW50 MX-NoLED, SW51 MX-NoLED, SW52 MX-NoLED, SW53 MX-NoLED, SW54 MX-NoLED, SW55 MX-NoLED, SW56 MX-NoLED, SW57 MX-NoLED, SW58 Reset, SW6 MX-NoLED, SW7 MX-NoLED, SW8 MX-NoLED, SW9 MX-NoLED, U1 ATmega32U4-AU, Y1 16MHz

Commit message: fix rows and start new traces
Connections:
- no-connect marks 9 -> 5
Changed lines of the file:
@@
 Text Label 3500 4500 0    50   ~ 0
 Col15
-NoConn ~ 3500 4700
-NoConn ~ 3500 4800
-NoConn ~ 3500 4900
-NoConn ~ 3500 5000
 $Comp
 L Device:C C8
@@
 Text Notes 12000 4450 0    63   ~ 0
 RGB LEDs
+Text Label 3500 4700 0    50   ~ 0
+Row1
+Text Label 3500 4800 0    50   ~ 0
+Row2
+Text Label 3500 4900 0    50   ~ 0
+Row3
+Text Label 3500 5000 0    50   ~ 0
+Row4
 $EndSCHEMATC

Commit message: rotary encoder?
Parts:
- added D53: 1N4148, orch:D_DO-35_SOD27_P5.08mm_Horizontal, symbol Device:D
- added SW53: Rotary_Encoder_Switch, Rotary_Encoder:RotaryEncoder_Alps_EC11E-Switch_Vertical_H20mm, symbol Device:Rotary_Encoder_Switch
- renumbered D53 to D54, D54 to D55, D55 to D56, D56 to D57, D57 to D58, D58 to D59, D59 to D60, D60 to D61, D61 to D62, D62 to D63, SW53 to SW54, SW54 to SW55, SW55 to SW56, SW56 to SW57, SW57 to SW58
Connections:
- net labels added: RotaryA, RotaryB
- wire segments 201 -> 204
Changed lines of the file:
@@
 $EndComp
 $Comp
-L orch:MX-NoLED SW53
+L orch:MX-NoLED SW54
 U 1 1 60176675
 P 14500 8850
-F 0 "SW53" V 14514 8978 60  0000 L CNN
+F 0 "SW54" V 14514 8978 60  0000 L CNN
 F 1 "MX-NoLED" V 14588 8978 20  0000 L CNN
 F 2 "orch:MX-1U-NoLED" H 13875 8825 60  0001 C CNN
@@
 $EndComp
 $Comp
-L Device:D D53
+L Device:D D54
 U 1 1 60177249
 P 14550 9150
-F 0 "D53" V 14596 9070 50  0000 R CNN
+F 0 "D54" V 14596 9070 50  0000 R CNN
 F 1 "1N4148" V 14505 9070 50  0000 R CNN
 F 2 "orch:D_DO-35_SOD27_P5.08mm_Horizontal" H 14550 9150 50  0001 C CNN
@@
 $EndComp
 $Comp
-L orch:MX-NoLED SW54
+L orch:MX-NoLED SW55
 U 1 1 6017D643
 P 15100 7050
-F 0 "SW54" V 15114 7178 60  0000 L CNN
+F 0 "SW55" V 15114 7178 60  0000 L CNN
 F 1 "MX-NoLED" V 15188 7178 20  0000 L CNN
 F 2 "orch:MX-1U-NoLED" H 14475 7025 60  0001 C CNN
@@
 $EndComp
 $Comp
-L Device:D D54
+L Device:D D55
 U 1 1 6017DB44
 P 15150 7350
-F 0 "D54" V 15196 7270 50  0000 R CNN
+F 0 "D55" V 15196 7270 50  0000 R CNN
 F 1 "1N4148" V 15105 7270 50  0000 R CNN
 F 2 "orch:D_DO-35_SOD27_P5.08mm_Horizontal" H 15150 7350 50  0001 C CNN
@@
 $EndComp
 $Comp
-L orch:MX-NoLED SW55
+L orch:MX-NoLED SW56
 U 1 1 6017DFBF
 P 15100 7650
-F 0 "SW55" V 15114 7778 60  0000 L CNN
+F 0 "SW56" V 15114 7778 60  0000 L CNN
 F 1 "MX-NoLED" V 15188 7778 20  0000 L CNN
 F 2 "orch:MX-1U-NoLED" H 14475 7625 60  0001 C CNN
@@
 $EndComp
 $Comp
-L Device:D D55
+L Device:D D56
 U 1 1 6017E5B4
 P 15150 7950
-F 0 "D55" V 15196 7870 50  0000 R CNN
+F 0 "D56" V 15196 7870 50  0000 R CNN
 F 1 "1N4148" V 15105 7870 50  0000 R CNN
 F 2 "orch:D_DO-35_SOD27_P5.08mm_Horizontal" H 15150 7950 50  0001 C CNN
@@
 $EndComp
 $Comp
-L orch:MX-NoLED SW56
+L orch:MX-NoLED SW57
 U 1 1 6017EB42
 P 15100 8250
-F 0 "SW56" V 15114 8378 60  0000 L CNN
+F 0 "SW57" V 15114 8378 60  0000 L CNN
 F 1 "MX-NoLED" V 15188 8378 20  0000 L CNN
 F 2 "orch:MX-1U-NoLED" H 14475 8225 60  0001 C CNN
@@
 $EndComp
 $Comp
-L Device:D D56
+L Device:D D57
 U 1 1 6017EF94
 P 15150 8550
-F 0 "D56" V 15196 8470 50  0000 R CNN
+F 0 "D57" V 15196 8470 50  0000 R CNN
 F 1 "1N4148" V 15105 8470 50  0000 R CNN
 F 2 "orch:D_DO-35_SOD27_P5.08mm_Horizontal" H 15150 8550 50  0001 C CNN
@@
 $EndComp
 $Comp
-L orch:MX-NoLED SW57
+L orch:MX-NoLED SW58
 U 1 1 6017F347
 P 15100 8850
-F 0 "SW57" V 15114 8978 60  0000 L CNN
+F 0 "SW58" V 15114 8978 60  0000 L CNN
 F 1 "MX-NoLED" V 15188 8978 20  0000 L CNN
 F 2 "orch:MX-1U-NoLED" H 14475 8825 60  0001 C CNN
@@
 $EndComp
 $Comp
-L Device:D D57
+L Device:D D58
 U 1 1 6017F9A6
 P 15150 9150
-F 0 "D57" V 15196 9070 50  0000 R CNN
+F 0 "D58" V 15196 9070 50  0000 R CNN
 F 1 "1N4148" V 15105 9070 50  0000 R CNN
 F 2 "orch:D_DO-35_SOD27_P5.08mm_Horizontal" H 15150 9150 50  0001 C CNN
@@
 Connection ~ 14350 7000
 $Comp
-L LED:SK6812 D60
+L LED:SK6812 D61
 U 1 1 60043709
 P 12200 5150
-F 0 "D60" H 12544 5196 50  0000 L CNN
+F 0 "D61" H 12544 5196 50  0000 L CNN
 F 1 "SK6812" H 12544 5105 50  0000 L CNN
 F 2 "LED_SMD:LED_SK6812_PLCC4_5.0x5.0mm_P3.2mm" H 12250 4850 50  0001 L TNN
@@
 $EndComp
 $Comp
-L LED:SK6812 D59
+L LED:SK6812 D60
 U 1 1 6004455E
 P 11150 5150
-F 0 "D59" H 11494 5196 50  0000 L CNN
+F 0 "D60" H 11494 5196 50  0000 L CNN
 F 1 "SK6812" H 11494 5105 50  0000 L CNN
 F 2 "LED_SMD:LED_SK6812_PLCC4_5.0x5.0mm_P3.2mm" H 11200 4850 50  0001 L TNN
@@
 $EndComp
 $Comp
-L LED:SK6812 D58
+L LED:SK6812 D59
 U 1 1 600451BB
 P 10100 5150
-F 0 "D58" H 10444 5196 50  0000 L CNN
+F 0 "D59" H 10444 5196 50  0000 L CNN
 F 1 "SK6812" H 10444 5105 50  0000 L CNN
 F 2 "LED_SMD:LED_SK6812_PLCC4_5.0x5.0mm_P3.2mm" H 10150 4850 50  0001 L TNN
@@
 $EndComp
 $Comp
-L LED:SK6812 D61
+L LED:SK6812 D62
 U 1 1 600459D4
 P 13250 5150
-F 0 "D61" H 13594 5196 50  0000 L CNN
+F 0 "D62" H 13594 5196 50  0000 L CNN
 F 1 "SK6812" H 13594 5105 50  0000 L CNN
 F 2 "LED_SMD:LED_SK6812_PLCC4_5.0x5.0mm_P3.2mm" H 13300 4850 50  0001 L TNN
@@
 $EndComp
 $Comp
-L LED:SK6812 D62
+L LED:SK6812 D63
 U 1 1 60047365
 P 14300 5150
-F 0 "D62" H 14644 5196 50  0000 L CNN
+F 0 "D63" H 14644 5196 50  0000 L CNN
 F 1 "SK6812" H 14644 5105 50  0000 L CNN
 F 2 "LED_SMD:LED_SK6812_PLCC4_5.0x5.0mm_P3.2mm" H 14350 4850 50  0001 L TNN
@@
 Text Label 3500 5000 0    50   ~ 0
 Row4
+$Comp
+L Device:Rotary_Encoder_Switch SW53
+U 1 1 601A2F6C
+P 7600 1850
+F 0 "SW53" H 7600 2217 50  0000 C CNN
+F 1 "Rotary_Encoder_Switch" H 7600 2126 50  0000 C CNN
+F 2 "Rotary_Encoder:RotaryEncoder_Alps_EC11E-Switch_Vertical_H20mm" H 7450 2010 50  0001 C CNN
+F 3 "~" H 7600 2110 50  0001 C CNN
+	1    7600 1850
+	1    0    0    -1
+$EndComp
+$Comp
+L Device:D D53
+U 1 1 601A60C9
+P 8050 2100
+F 0 "D53" V 8096 2020 50  0000 R CNN
+F 1 "1N4148" V 8005 2020 50  0000 R CNN
+F 2 "orch:D_DO-35_SOD27_P5.08mm_Horizontal" H 8050 2100 50  0001 C CNN
+F 3 "~" H 8050 2100 50  0001 C CNN
+	1    8050 2100
+	0    -1   -1   0
+$EndComp
+Wire Wire Line
+	7900 1950 8050 1950
+Text Label 8050 2250 3    50   ~ 0
+Row3
+Text Label 7900 1750 0    50   ~ 0
+Col14
+$Comp
+L power:GND #PWR?
+U 1 1 601B43AD
+P 6950 2100
+F 0 "#PWR?" H 6950 1850 50  0001 C CNN
+F 1 "GND" H 6955 1927 50  0000 C CNN
+F 2 "" H 6950 2100 50  0001 C CNN
+F 3 "" H 6950 2100 50  0001 C CNN
+	1    6950 2100
+	1    0    0    -1
+$EndComp
+Wire Wire Line
+	7300 1850 6950 1850
+Wire Wire Line
+	6950 1850 6950 2100
+Text Label 7300 1750 2    50   ~ 0
+RotaryA
+Text Label 7300 1950 2    50   ~ 0
+RotaryB
 $EndSCHEMATC

Commit message: v2!
Parts:
- added D25, D29: 1N4148, orch:D_DO-35_SOD27_P5.08mm_Horizontal, symbol Device:D
- added D66: SK6812, LED_SMD:LED_SK6812_PLCC4_5.0x5.0mm_P3.2mm, symbol LED:SK6812
- added SW25: MX-NoLED, orch:MX-2U-NoLED, symbol orch:MX-NoLED
- added SW29: MX-NoLED, orch:MX-1U-NoLED, symbol orch:MX-NoLED
- SW24: footprint orch:MX-2U-NoLED -> orch:MX-1U-NoLED
- SW51: renamed from SW49; footprint orch:MX-2.25U-NoLED -> orch:MX-1.75U-NoLED
- SW55: renamed from SW53; footprint Rotary_Encoder:RotaryEncoder_Alps_EC11E-Switch_Vertical_H20mm -> orch:RotaryEncoder_Alps_EC11E-Switch_Vertical_H20mm
- renumbered D25 to D26, D26 to D27, D27 to D28, D28 to D30, D29 to D31, D30 to D32, D31 to D33, D32 to D34, D33 to D35, D34 to D36, D35 to D37, D36 to D38, D37 to D39, D38 to D40, D39 to D41, D40 to D42, D41 to D43, D42 to D44, D43 to D45, D44 to D46, D45 to D47, D46 to D48, D47 to D49, D48 to D50, D49 to D51, D50 to D52, D51 to D53, D52 to D54, D53 to D55, D54 to D56, D55 to D57, D56 to D58, D57 to D59, D58 to D60, D59 to D61, D60 to D62, D61 to D63, D62 to D64, D63 to D65, SW25 to SW26, SW26 to SW27, SW27 to SW28, SW28 to SW30, SW29 to SW31, SW30 to SW32, SW31 to SW33, SW32 to SW34, SW33 to SW35, SW34 to SW36, SW35 to SW37, SW36 to SW38, SW37 to SW39, SW38 to SW40, SW39 to SW41, SW40 to SW42, SW41 to SW43, SW42 to SW44, SW43 to SW45, SW44 to SW46, SW45 to SW47, SW46 to SW48, SW47 to SW49, SW48 to SW50, SW50 to SW52, SW51 to SW53, SW52 to SW54, SW54 to SW56, SW55 to SW57, SW56 to SW58, SW57 to SW59, SW58 to SW60, SW58 to SW61
Connections:
- wire segments 204 -> 213
- no-connect marks 5 -> 3
Other:
- note added: "Rotary Encoder"

Commit message: some new case things, updated BOM
Connections:
- wire segments 213 -> 214
Changed lines of the file:
@@
 	8700 4000 8300 4000
 Wire Wire Line
-	8000 3700 7750 3700
-Wire Wire Line
-	7750 3700 7750 3600
-Wire Wire Line
 	8000 4000 7750 4000
-Wire Wire Line
-	7750 4000 7750 3700
-Connection ~ 7750 3700
 Wire Wire Line
 	8700 3700 8300 3700
@@
 L power:GND #PWR05
 U 1 1 5F122095
-P 7750 3600
-F 0 "#PWR05" H 7750 3350 50  0001 C CNN
-F 1 "GND" H 7755 3427 50  0000 C CNN
-F 2 "" H 7750 3600 50  0001 C CNN
-F 3 "" H 7750 3600 50  0001 C CNN
-	1    7750 3600
-	-1   0    0    1
+P 7750 4450
+F 0 "#PWR05" H 7750 4200 50  0001 C CNN
+F 1 "GND" H 7755 4277 50  0000 C CNN
+F 2 "" H 7750 4450 50  0001 C CNN
+F 3 "" H 7750 4450 50  0001 C CNN
+	1    7750 4450
+	1    0    0    -1
 $EndComp
 $Comp
@@
 Wire Wire Line
 	7900 1950 8050 1950
-Text Label 8050 2250 3    50   ~ 0
+Text Label 8050 2450 0    50   ~ 0
 Row3
 Text Label 7900 1750 0    50   ~ 0
@@
 Text Notes 7250 1250 0    63   ~ 0
 Rotary Encoder
+Wire Wire Line
+	8000 3700 7750 3700
+Wire Wire Line
+	7750 3700 7750 4000
+Connection ~ 7750 4000
+Wire Wire Line
+	7750 4000 7750 4450
+Wire Wire Line
+	8050 2250 8050 2450
 $EndSCHEMATC

Commit message: fix caps for leds
Parts:
- added C10, C11, C12, C13, C14, C9: 0.1u, Capacitor_SMD:C_0805_2012Metric_Pad1.15x1.40mm_HandSolder, symbol Device:C
Connections:
- wire segments 214 -> 238

Commit message: v2.1 - add caps to LEDs, re-do some routing
Parts:
- renumbered R3 to R2, R2 to R3
Changed lines of the file:
@@
 Title "orch"
 Date ""
-Rev "v2"
+Rev "v2.1"
 Comp ""
 Comment1 ""
@@
 Reset
 $Comp
-L Device:R R2
+L Device:R R3
 U 1 1 6005B30E
 P 12700 2500
-F 0 "R2" V 12493 2500 50  0000 C CNN
+F 0 "R3" V 12493 2500 50  0000 C CNN
 F 1 "22R" V 12584 2500 50  0000 C CNN
 F 2 "Resistor_SMD:R_0805_2012Metric_Pad1.15x1.40mm_HandSolder" V 12630 2500 50  0001 C CNN
@@
 D-
 $Comp
-L Device:R R3
+L Device:R R2
 U 1 1 600600F3
 P 12700 2700
-F 0 "R3" V 12907 2700 50  0000 C CNN
+F 0 "R2" V 12907 2700 50  0000 C CNN
 F 1 "22R" V 12816 2700 50  0000 C CNN
 F 2 "Resistor_SMD:R_0805_2012Metric_Pad1.15x1.40mm_HandSolder" V 12630 2700 50  0001 C CNN

Commit message: update bom, renumber caps
Parts:
- renumbered C11 to C10, C12 to C11, C13 to C12, C14 to C13, C8 to C14, C9 to C8, C10 to C9
Changed lines of the file:
@@
 Col15
 $Comp
-L Device:C C8
+L Device:C C14
 U 1 1 603A0FBA
 P 2100 3550
-F 0 "C8" H 1985 3504 50  0000 R CNN
+F 0 "C14" H 1985 3504 50  0000 R CNN
 F 1 "1u" H 1985 3595 50  0000 R CNN
 F 2 "Capacitor_SMD:C_0805_2012Metric_Pad1.15x1.40mm_HandSolder" H 2138 3400 50  0001 C CNN
@@
 	8050 2250 8050 2450
 $Comp
-L Device:C C9
+L Device:C C8
 U 1 1 60244178
 P 9900 4700
-F 0 "C9" H 9785 4654 50  0000 R CNN
+F 0 "C8" H 9785 4654 50  0000 R CNN
 F 1 "0.1u" H 9785 4745 50  0000 R CNN
 F 2 "Capacitor_SMD:C_0805_2012Metric_Pad1.15x1.40mm_HandSolder" H 9938 4550 50  0001 C CNN
@@
 	10200 5450 10550 5450
 $Comp
-L Device:C C10
+L Device:C C9
 U 1 1 60290B28
 P 10950 4700
-F 0 "C10" H 10835 4654 50  0000 R CNN
+F 0 "C9" H 10835 4654 50  0000 R CNN
 F 1 "0.1u" H 10835 4745 50  0000 R CNN
 F 2 "Capacitor_SMD:C_0805_2012Metric_Pad1.15x1.40mm_HandSolder" H 10988 4550 50  0001 C CNN
@@
 	11250 5450 11600 5450
 $Comp
-L Device:C C11
+L Device:C C10
 U 1 1 6029EA5A
 P 12000 4700
-F 0 "C11" H 11885 4654 50  0000 R CNN
+F 0 "C10" H 11885 4654 50  0000 R CNN
 F 1 "0.1u" H 11885 4745 50  0000 R CNN
 F 2 "Capacitor_SMD:C_0805_2012Metric_Pad1.15x1.40mm_HandSolder" H 12038 4550 50  0001 C CNN
@@
 	12300 5450 12650 5450
 $Comp
-L Device:C C12
+L Device:C C11
 U 1 1 602AD2FE
 P 13050 4700
-F 0 "C12" H 12935 4654 50  0000 R CNN
+F 0 "C11" H 12935 4654 50  0000 R CNN
 F 1 "0.1u" H 12935 4745 50  0000 R CNN
 F 2 "Capacitor_SMD:C_0805_2012Metric_Pad1.15x1.40mm_HandSolder" H 13088 4550 50  0001 C CNN
@@
 	13350 5450 13700 5450
 $Comp
-L Device:C C13
+L Device:C C12
 U 1 1 602BC21C
 P 14100 4700
-F 0 "C13" H 13985 4654 50  0000 R CNN
+F 0 "C12" H 13985 4654 50  0000 R CNN
 F 1 "0.1u" H 13985 4745 50  0000 R CNN
 F 2 "Capacitor_SMD:C_0805_2012Metric_Pad1.15x1.40mm_HandSolder" H 14138 4550 50  0001 C CNN
@@
 	14400 5450 14750 5450
 $Comp
-L Device:C C14
+L Device:C C13
 U 1 1 602E26CF
 P 15150 4700
-F 0 "C14" H 15035 4654 50  0000 R CNN
+F 0 "C13" H 15035 4654 50  0000 R CNN
 F 1 "0.1u" H 15035 4745 50  0000 R CNN
 F 2 "Capacitor_SMD:C_0805_2012Metric_Pad1.15x1.40mm_HandSolder" H 15188 4550 50  0001 C CNN
