File: pcb/orch.sch (KiCad schematic (older format))
At the start: 152 parts, among them J1 AVR-ISP-6, P1 USB_C_Receptacle_USB2.0, SW1 MX-NoLED, SW10 MX-NoLED, SW11 MX-NoLED, SW12 MX-NoLED, SW13 MX-NoLED, SW14 MX-NoLED, SW15 MX-NoLED, SW16 MX-NoLED, SW17 MX-NoLED, SW18 MX-NoLED, SW19 MX-NoLED, SW2 MX-NoLED, SW20 MX-NoLED, SW21 MX-NoLED, SW22 MX-NoLED, SW23 MX-NoLED, SW24 MX-NoLED, SW25 MX-NoLED, SW26 MX-NoLED, SW27 MX-NoLED, SW28 MX-NoLED, SW29 MX-NoLED, SW3 MX-NoLED, SW30 MX-NoLED, SW31 MX-NoLED, SW32 MX-NoLED, SW33 MX-NoLED, SW34 MX-NoLED, SW35 MX-NoLED, SW36 MX-NoLED, SW37 MX-NoLED, SW38 MX-NoLED, SW39 MX-NoLED, SW4 MX-NoLED, SW40 MX-NoLED, SW41 MX-NoLED, SW42 MX-NoLED, SW43 MX-NoLED, SW44 MX-NoLED, SW45 MX-NoLED, SW46 MX-NoLED, SW47 MX-NoLED, SW48 MX-NoLED, SW49 MX-NoLED, SW5 MX-NoLED, SW50 MX-NoLED, SW51 MX-NoLED, SW52 MX-NoLED, SW53 MX-NoLED, SW54 MX-NoLED, SW55 Rotary_Encoder_Switch, SW56 MX-NoLED, SW57 MX-NoLED, SW58 MX-NoLED, SW59 MX-NoLED, SW6 MX-NoLED, SW60 MX-NoLED, SW61 Reset, SW7 MX-NoLED, SW8 MX-NoLED, SW9 MX-NoLED, U1 ATmega32U4-AU, Y1 16MHz

Commit message: ?
Parts:
- P1: symbol Connector:USB_C_Receptacle_USB2.0 -> orch-rescue:USB_C_Receptacle_USB2.0-Connector
Changed lines of the file:
@@
 $EndComp
 $Comp
-L Connector:USB_C_Receptacle_USB2.0 P1
+L orch-rescue:USB_C_Receptacle_USB2.0-Connector P1
 U 1 1 5F152268
 P 11500 2600

Commit message: + wip
Parts:
- removed C10, C11, C12, C13, C8, C9: 0.1u, Capacitor_SMD:C_0805_2012Metric_Pad1.15x1.40mm_HandSolder, symbol Device:C
- removed D61, D62, D63, D64, D65, D66: SK6812, LED_SMD:LED_SK6812_PLCC4_5.0x5.0mm_P3.2mm, symbol LED:SK6812
- added D61, D62, D63, D64, D65, D66, D67, D68, D69, D70, D71, D72, D73, D74, D75: 1N4148, orch:D_DO-35_SOD27_P5.08mm_Horizontal, symbol Device:D
- added SW61, SW62, SW63, SW64, SW65, SW66, SW67, SW68, SW69, SW70, SW71, SW72, SW73, SW75: MX-NoLED, orch:MX-1U-NoLED, symbol orch:MX-NoLED
- added SW74: MX-NoLED, orch:MX-1.5U-NoLED, symbol orch:MX-NoLED
- renumbered SW61 to SW76
Connections:
- net labels added: Row5, USB_D+, USB_D-
- wire segments 238 -> 228
Other:
- note removed: "RGB LEDs"

Commit message: re-add LEDs
Parts:
- added C10, C11, C12, C13, C14, C15, C16, C9: 0.1u, Capacitor_SMD:C_0805_2012Metric_Pad1.18x1.45mm_HandSolder, symbol Device:C
- added D76, D77, D78, D79, D80, D81, D82, D83: SK6812, LED_SMD:LED_SK6812_PLCC4_5.0x5.0mm_P3.2mm, symbol LED:SK6812
- C1, C2, C3, C4, C5, C6, C7: footprint Capacitor_SMD:C_0805_2012Metric_Pad1.15x1.40mm_HandSolder -> Capacitor_SMD:C_0805_2012Metric_Pad1.18x1.45mm_HandSolder
- C8: renamed from C14; footprint Capacitor_SMD:C_0805_2012Metric_Pad1.15x1.40mm_HandSolder -> Capacitor_SMD:C_0805_2012Metric_Pad1.18x1.45mm_HandSolder
Connections:
- wire segments 228 -> 283
- no-connect marks 3 -> 4
Other:
- note added: "RGB LEDs"

Commit message: v1?
Parts:
- SW48: footprint orch:MX-1.25U-NoLED -> orch:MX-1U-NoLED
Changed lines of the file:
@@
 Text Label 3500 2300 0    50   ~ 0
 MOSI
-Text Label 3800 2400 0    50   ~ 0
+Text Label 3500 2400 0    50   ~ 0
 MISO
 Text Label 3500 2200 0    50   ~ 0
@@
 F 0 "SW48" V 13314 8878 60  0000 L CNN
 F 1 "MX-NoLED" V 13388 8878 20  0000 L CNN
-F 2 "orch:MX-1.25U-NoLED" H 12675 8725 60  0001 C CNN
+F 2 "orch:MX-1U-NoLED" H 12675 8725 60  0001 C CNN
 F 3 "" H 12675 8725 60  0001 C CNN
 	1    13300 8750
@@
 Text Label 14950 6750 1    50   ~ 0
 Col15
-Text Label 3500 2400 0    50   ~ 0
+Text Label 3800 2300 0    50   ~ 0
 Row1
 $Comp
@@
 Text Label 3500 4800 0    50   ~ 0
 RGB
-Wire Wire Line
-	3500 2400 3800 2400
 $Comp
 L LED:SK6812 D76
@@
 Text Notes 11350 4850 0    63   ~ 0
 RGB LEDs
+Wire Wire Line
+	3500 2300 3800 2300
 $EndSCHEMATC

Commit message: Fix key
Parts:
- removed D25: 1N4148, orch:D_DO-35_SOD27_P5.08mm_Horizontal, symbol Device:D
- SW74: footprint orch:MX-1.5U-NoLED -> orch:MX-1U-NoLED
Connections:
- net labels added: SW25
- wire segments 283 -> 280
Changed lines of the file:
@@
 	9150 9800 9750 9800
 Connection ~ 9750 9800
-Wire Wire Line
-	9750 9800 10150 9800
 Connection ~ 10950 9800
 Wire Wire Line
@@
 	0    1    1    0
 $EndComp
-$Comp
-L Device:D D25
-U 1 1 60238050
-P 9750 10250
-F 0 "D25" V 9796 10170 50  0000 R CNN
-F 1 "1N4148" V 9705 10170 50  0000 R CNN
-F 2 "orch:D_DO-35_SOD27_P5.08mm_Horizontal" H 9750 10250 50  0001 C CNN
-F 3 "~" H 9750 10250 50  0001 C CNN
-	1    9750 10250
-	0    -1   -1   0
-$EndComp
 Wire Wire Line
 	9550 9300 9550 9900
 Connection ~ 9550 9300
-Wire Wire Line
-	9750 10400 10150 10400
-Wire Wire Line
-	10150 10400 10150 9800
-Connection ~ 10150 9800
-Wire Wire Line
-	10150 9800 10350 9800
 Text Label 3500 4700 0    50   ~ 0
 RotaryA
@@
 F 0 "SW74" V 14514 7078 60  0000 L CNN
 F 1 "MX-NoLED" V 14588 7078 20  0000 L CNN
-F 2 "orch:MX-1.5U-NoLED" H 13875 6925 60  0001 C CNN
+F 2 "orch:MX-1U-NoLED" H 13875 6925 60  0001 C CNN
 F 3 "" H 13875 6925 60  0001 C CNN
 	1    14500 6950
@@
 Wire Wire Line
 	3500 2300 3800 2300
+Text Label 9750 9500 0    50   ~ 0
+SW25
+Text Label 9750 10100 3    50   ~ 0
+SW25
+Wire Wire Line
+	9750 9800 10350 9800
 $EndSCHEMATC
